Commit message: feat(ros2_quadruped_kit): complete verification, hardware firmware, emulator, and tests for Milestone 5.4
- Fix xacro stderr duplicate pi declaration in quadruped.urdf.xacro
- Fix empty ros__parameters block in ros2_controllers.yaml preventing rcl crash
- Add serial_port xacro parameterization and ParameterValue string wrapping
- Add IMU topic remapping in hardware.launch.py to seamlessly feed state estimator
- Add physical Arduino firmware sketch (arduino/quadruped_controller/quadruped_controller.ino) with 12-actuator torque/position streaming and IMU telemetry
- Add desktop virtual PTY hardware emulator (scripts/pseudo_quadruped_emulator.py)
- Add comprehensive automated verification test suite (scripts/test_quadruped_kit.py) testing kinematics, dynamics, estimators, ros2_control, demos, and breakers
- Update kit README and pedagogical articles (LEG 02, LEG 15) with firmware and emulation references

File: Ros2 learning kits/ros2_quadruped_kit/src/quadruped_description/urdf/quadruped.urdf.xacro (robot description, xacro)
@@ -15,6 +15,4 @@
   <!-- Include macros -->
   <xacro:include filename="$(find quadruped_description)/urdf/leg_macro.urdf.xacro"/>
-  <!-- Constants -->
-  <xacro:property name="pi" value="3.14159265359"/>
   <!-- Body dimensions -->
   <xacro:property name="body_length" value="0.40"/>
@@ -25,4 +23,5 @@
   <xacro:arg name="use_sim" default="false"/>
   <xacro:arg name="use_fake_hardware" default="false"/>
+  <xacro:arg name="serial_port" default="/dev/ttyUSB0"/>
   <!-- ==================== BASE LINK ==================== -->
   <link name="base_link">
@@ -123,5 +122,5 @@
         <hardware>
           <plugin>quadruped_hardware/LegHardwareInterface</plugin>
-          <param name="serial_port">/dev/ttyUSB0</param>
+          <param name="serial_port">$(arg serial_port)</param>
           <param name="baud_rate">1000000</param>
         </hardware>
